Commit message: limit追加

File: universal_robot/ur_description/urdf/ur3_joint_limited_robot.urdf.xacro (robot description, xacro)
@@ -6,4 +6,5 @@
   <!-- ur3 -->
   <xacro:include filename="$(find ur_description)/urdf/ur3.urdf.xacro" />
+    <xacro:include filename="$(find realsense2_description)/urdf/test_d415_camera.urdf.xacro" />
   <!-- arm -->
   <xacro:ur3_robot prefix="" joint_limited="true"
@@ -19,5 +20,18 @@
     <parent link="world" />
     <child link = "base_link" />
-    <origin xyz="0.0 0.0 0.0" rpy="0.0 0.0 0.0" />
+    <origin xyz="0.0 0.0 0.04" rpy="0.0 0.0 0.0" />
   </joint>
+      <joint name="ommc_joint" type="fixed">
+      <parent link="world" />
+      <child link = "thin_link" />
+      <origin xyz="-0.5 0.0 0.0" rpy="0.0 0.0 0.0" />
+    </joint>
+    <link name="thin_link">
+      <collision>
+        <geometry>
+          <box size="0.01 0.01 0.01"/>
+        </geometry>
+        <origin rpy="00 0 0" xyz="0 0 0"/>
+      </collision>
+    </link>
 </robot>
