Commit message: mody追加

File: universal_robot/ur_description/urdf/ur3.urdf.xacro (robot description, xacro)
@@ -1,4 +1,4 @@
 <?xml version="1.0"?>
-<robot xmlns:xacro="http://wiki.ros.org/xacro">
+<robot xmlns:xacro="http://ros.org/wiki/xacro">
 <!--
   Author: Felix Messmer
@@ -16,11 +16,10 @@
   </xacro:macro>
   <xacro:macro name="ur3_robot" params="prefix joint_limited
-    shoulder_pan_lower_limit:=${-pi}    shoulder_pan_upper_limit:=${pi}
-    shoulder_lift_lower_limit:=${-pi}    shoulder_lift_upper_limit:=${pi}
-    elbow_joint_lower_limit:=${-pi}    elbow_joint_upper_limit:=${pi}
-    wrist_1_lower_limit:=${-pi}    wrist_1_upper_limit:=${pi}
-    wrist_2_lower_limit:=${-pi}    wrist_2_upper_limit:=${pi}
-    wrist_3_lower_limit:=${-pi}    wrist_3_upper_limit:=${pi}
-    transmission_hw_interface:=hardware_interface/PositionJointInterface">
+     shoulder_pan_lower_limit:=${-pi}    shoulder_pan_upper_limit:=${pi}
+     shoulder_lift_lower_limit:=${-pi}    shoulder_lift_upper_limit:=${pi}
+     elbow_joint_lower_limit:=${-pi}    elbow_joint_upper_limit:=${pi}
+     wrist_1_lower_limit:=${-pi}    wrist_1_upper_limit:=${pi}
+     wrist_2_lower_limit:=${-pi}    wrist_2_upper_limit:=${pi}
+     wrist_3_lower_limit:=${-pi}    wrist_3_upper_limit:=${pi}">
     <!-- Inertia parameters -->
     <xacro:property name="base_mass" value="2.0" />  <!-- This mass might be incorrect -->
@@ -74,5 +73,5 @@
       </collision>
       <xacro:cylinder_inertial radius="0.075" length="0.038" mass="${base_mass}">
-        <origin xyz="0.0 0.0 0.0" rpy="0 0 0" />
+        <origin xyz="0.0 0.0 0.04" rpy="0 0 0" />
       </xacro:cylinder_inertial>
     </link>
@@ -265,21 +264,122 @@
     <joint name="${prefix}ee_fixed_joint" type="fixed">
       <parent link="${prefix}wrist_3_link" />
+      <child link = "${prefix}ee_link" />
+      <origin xyz="0.0 0.23101 0.0" rpy="${pi/2.0} ${pi/2.0} ${pi/2.0}" />
+    </joint>
+    <!-- <link name="${prefix}ee_link">
+    <visual>
+        <geometry>
+          <mesh filename="package://ur_description/meshes/ur3/visual/osd.stl"/>
+        </geometry>
+        <material name="LightGrey">
+          <color rgba="0.8 0.8 0.8 1.0"/>
+        </material>
+    </visual>
+      <collision>
+        <geometry>
+          <mesh filename="package://ur_description/meshes/ur3/visual/osd.stl"/>
+        </geometry>
+        <origin rpy="0 0 0" xyz="-0.015 0.135 0"/>
+        </collision>
+    </link> -->
+    <link name="${prefix}ee_link">
+      <collision>
+        <geometry>
+          <box size="0.01 0.01 0.01"/>
+        </geometry>
+        <origin rpy="0 0 0" xyz="-0.01 0 0"/>
+      </collision>
+      <material name="LightGrey">
+          <color rgba="0.7 0.7 0.7 1.0"/>
+      </material>
+    </link>
+    <joint name="${prefix}camera_fixed_joint" type="fixed">
+      <parent link="${prefix}wrist_3_link" />
+      <child link = "${prefix}camerass_link" />
+      <origin xyz="-0.02 0.12443 0.0293" rpy="${0} ${0} ${pi/2}" />
+    </joint>
+    <link name="${prefix}camerass_link">
+      <collision>
+        <geometry>
+          <box size="0.01 0.01 0.01"/>
+        </geometry>
+        <origin rpy="00 0 0" xyz="0 0 0"/>
+      </collision>
+    </link>
+    <joint name="${prefix}force_jyoint" type="fixed">
+      <parent link="${prefix}wrist_3_link" />
+      <child link = "${prefix}force_mount_link" />
+      <origin xyz="0 ${wrist_3_length} 0" rpy="${0} ${pi/2} ${pi/2}" />
+    </joint>
+    <link name="${prefix}force_mount_link">
+    <visual>
+        <geometry>
+          <mesh filename="package://ur_description/meshes/ur3/visual/force_mount.stl"/>
+        </geometry>
+        <material name="Light_Blue">
+          <color rgba="0.0 1.0 1.0 1.0"/>
+        </material>
+    </visual>
+      <collision>
+        <geometry>
+          <mesh filename="package://ur_description/meshes/ur3/visual/force_mount.stl"/>
+        </geometry>
+        <origin rpy="0 0 0" xyz="0 0 0"/>
+        </collision>
+    </link>
+        <joint name="${prefix}force_top_joy" type="fixed">
+      <parent link="${prefix}force_mount_link" />
+      <child link = "${prefix}force_top_link" />
+      <origin xyz="${0} ${0} ${0.008}" rpy="${0} ${0} ${0}" />
+    </joint>
+    <link name="${prefix}force_top_link">
+    <visual>
+        <geometry>
+          <mesh filename="package://ur_description/meshes/ur3/visual/dynpick.stl"/>
+        </geometry>
+        <material name="red">
+          <color rgba="0.5 0.0 0.0 1.0"/>
+        </material>
+    </visual>
+      <collision>
+        <geometry>
+          <mesh filename="package://ur_description/meshes/ur3/visual/dynpick.stl"/>
+        </geometry>
+        <origin rpy="0 0 ${0}" xyz="0 0 0"/>
+        </collision>
+    </link>
+    <joint name="${prefix}camera_mount_joy" type="fixed">
+      <parent link="${prefix}force_top_link" />
+      <child link = "${prefix}camera_mount_link" />
+      <origin xyz="${0} ${0} ${0.0325}" rpy="${0} ${0} ${pi}" />
+    </joint>
+    <link name="${prefix}camera_mount_link">
+    <visual>
+        <geometry>
+          <mesh filename="package://ur_description/meshes/ur3/visual/cameramout.stl"/>
+        </geometry>
+        <material name="Light_Blue">
+          <color rgba="0.0 1.0 1.0 1.0"/>
+        </material>
+    </visual>
+      <collision>
+        <geometry>
+          <mesh filename="package://ur_description/meshes/ur3/visual/cameramout.stl"/>
+        </geometry>
+        <origin rpy="0 0 ${0}" xyz="0 0 0"/>
+        </collision>
+    </link>
+    <joint name="${prefix}robotiq_fixed_joint" type="fixed">
+      <parent link="${prefix}camera_mount_link" />
       <child link = "${prefix}robotiq_arg2f_base_link" />
-      <origin xyz="0.0 ${wrist_3_length} 0.0" rpy="0.0 ${pi/2.0} ${pi/2.0}" />
-    </joint>
-    <!-- <joint name="${prefix}ee_fixed_joint" type="fixed">
-      <parent link="${prefix}wrist_3_link" />
-      <child link = "${prefix}ee_link" />
-      <origin xyz="0.0 ${wrist_3_length} 0.0" rpy="0.0 0.0 ${pi/2.0}" />
-    </joint> -->
-    <!-- <link name="${prefix}ee_link">
-      <collision>
-        <geometry>
-          <box size="0.01 0.01 0.01"/>
-        </geometry>
-        <origin rpy="0 0 0" xyz="-0.01 0 0"/>
-      </collision>
-    </link> -->
-    <xacro:ur_arm_transmission prefix="${prefix}" hw_interface="${transmission_hw_interface}" />
+      <origin xyz="${0.0} ${0.0} ${0.025}" rpy="0.0 ${0.0} ${0.0}" />
+    </joint>
+    <joint name="${prefix}realsence_base_joint" type="fixed">
+      <parent link="${prefix}camera_mount_link" />
+      <child link = "${prefix}camera_base_link" />
+      <!-- z= 0.008+0.01018-->
+      <origin xyz="${0.055} ${0.0} ${0.01818}" rpy="${pi} ${3*pi/2.0} ${0}" />
+    </joint>
+    <xacro:ur_arm_transmission prefix="${prefix}" />
     <xacro:ur_arm_gazebo prefix="${prefix}" />
     <!-- ROS base_link to UR 'Base' Coordinates transform -->

File: universal_robot/ur_description/urdf/ur3_robot.urdf.xacro (robot description, xacro)
@@ -1,20 +1,33 @@
 <?xml version="1.0"?>
-<robot xmlns:xacro="http://wiki.ros.org/xacro"
+<robot xmlns:xacro="http://ros.org/wiki/xacro"
        name="ur3" >
-  <xacro:arg name="transmission_hw_interface" default="hardware_interface/PositionJointInterface"/>
   <!-- common stuff -->
   <xacro:include filename="$(find ur_description)/urdf/common.gazebo.xacro" />
   <!-- ur3 -->
   <xacro:include filename="$(find ur_description)/urdf/ur3.urdf.xacro" />
-  <xacro:include filename="$(find ur_description)/urdf/robotiq_arg2f_85_model.xacro" />
+  <!-- gripper -->
+  <xacro:include filename="$(find robotiq_2f_85_gripper_visualization)/urdf/robotiq_arg2f_85_model.xacro" />
+  <!-- realsense_model -->
+  <xacro:include filename="$(find realsense2_description)/urdf/test_d415_camera.urdf.xacro" />
   <!-- arm -->
-  <xacro:ur3_robot prefix="" joint_limited="false"
-    transmission_hw_interface="$(arg transmission_hw_interface)"
-  />
+  <xacro:ur3_robot prefix="" joint_limited="false"/>
   <link name="world" />
   <joint name="world_joint" type="fixed">
     <parent link="world" />
     <child link = "base_link" />
-    <origin xyz="0.0 0.0 0.0" rpy="0.0 0.0 0.0" />
+    <origin xyz="0.0 0.0 0.04" rpy="0.0 0.0 0.0" />
   </joint>
+      <joint name="ommc_joint" type="fixed">
+      <parent link="world" />
+      <child link = "thin_link" />
+      <origin xyz="-0.5 0.0 0.0" rpy="0.0 0.0 0.0" />
+    </joint>
+    <link name="thin_link">
+      <collision>
+        <geometry>
+          <box size="0.01 0.01 0.01"/>
+        </geometry>
+        <origin rpy="00 0 0" xyz="0 0 0"/>
+      </collision>
+    </link>
 </robot>

Commit message: ur3_robotiq_moveit_configで動く？

File: universal_robot/ur_description/urdf/ur3.urdf.xacro (robot description, xacro)
@@ -373,6 +373,22 @@
       <parent link="${prefix}camera_mount_link" />
       <child link = "${prefix}robotiq_arg2f_base_link" />
-      <origin xyz="${0.0} ${0.0} ${0.025}" rpy="0.0 ${0.0} ${0.0}" />
-    </joint>
+      <origin xyz="${0.0} ${0.0} ${0.008}" rpy="0.0 ${0.0} ${pi/2.0}" />
+    </joint>
+    <link name="${prefix}robotiq_arg2f_base_link">
+    <visual>
+        <geometry>
+          <mesh filename="package://ur_description/meshes/ur3/visual/hando_model.stl"/>
+        </geometry>
+        <material name="Light">
+          <color rgba="0.96875 0.70703125 0.0 1.0"/>
+        </material>
+    </visual>
+      <collision>
+        <geometry>
+          <mesh filename="package://ur_description/meshes/ur3/visual/hando_model.stl"/>
+        </geometry>
+        <origin rpy="0 0 ${0}" xyz="0 0 0"/>
+        </collision>
+    </link>
     <joint name="${prefix}realsence_base_joint" type="fixed">
       <parent link="${prefix}camera_mount_link" />

File: universal_robot/ur_description/urdf/ur3_robot.urdf.xacro (robot description, xacro)
@@ -7,5 +7,5 @@
   <xacro:include filename="$(find ur_description)/urdf/ur3.urdf.xacro" />
   <!-- gripper -->
-  <xacro:include filename="$(find robotiq_2f_85_gripper_visualization)/urdf/robotiq_arg2f_85_model.xacro" />
+  <!-- <xacro:include filename="$(find robotiq_2f_85_gripper_visualization)/urdf/robotiq_arg2f_85_model.xacro" /> -->
   <!-- realsense_model -->
   <xacro:include filename="$(find realsense2_description)/urdf/test_d415_camera.urdf.xacro" />

Commit message: ee_link_longver

File: universal_robot/ur_description/urdf/ur3.urdf.xacro (robot description, xacro)
@@ -263,24 +263,10 @@
     </link>
     <joint name="${prefix}ee_fixed_joint" type="fixed">
-      <parent link="${prefix}wrist_3_link" />
+      <parent link="${prefix}force_mount_link" />
       <child link = "${prefix}ee_link" />
-      <origin xyz="0.0 0.23101 0.0" rpy="${pi/2.0} ${pi/2.0} ${pi/2.0}" />
-    </joint>
-    <!-- <link name="${prefix}ee_link">
-    <visual>
-        <geometry>
-          <mesh filename="package://ur_description/meshes/ur3/visual/osd.stl"/>
-        </geometry>
-        <material name="LightGrey">
-          <color rgba="0.8 0.8 0.8 1.0"/>
-        </material>
-    </visual>
-      <collision>
-        <geometry>
-          <mesh filename="package://ur_description/meshes/ur3/visual/osd.stl"/>
-        </geometry>
-        <origin rpy="0 0 0" xyz="-0.015 0.135 0"/>
-        </collision>
-    </link> -->
+      <!-- <origin xyz="0.0 0.0 0.212242" rpy="${pi} 0 ${-pi/2.0} " /> -->
+      <!-- close +12mm -->
+      <origin xyz="0.0 0.0 0.224242" rpy="${pi} 0 ${-pi/2.0} " />
+    </joint>
     <link name="${prefix}ee_link">
       <collision>
@@ -290,12 +276,9 @@
         <origin rpy="0 0 0" xyz="-0.01 0 0"/>
       </collision>
-      <material name="LightGrey">
-          <color rgba="0.7 0.7 0.7 1.0"/>
-      </material>
     </link>
     <joint name="${prefix}camera_fixed_joint" type="fixed">
       <parent link="${prefix}wrist_3_link" />
       <child link = "${prefix}camerass_link" />
-      <origin xyz="-0.02 0.12443 0.0293" rpy="${0} ${0} ${pi/2}" />
+      <origin xyz="-0.02 0.12443 0.0293" rpy="${0} ${0} ${pi/2.0}" />
     </joint>
     <link name="${prefix}camerass_link">
@@ -307,4 +290,22 @@
       </collision>
     </link>
+    <!--
+    <link name="${prefix}ee_link">
+    <visual>
+        <geometry>
+          <mesh filename="package://ur_description/meshes/ur3/visual/osd.stl"/>
+        </geometry>
+        <material name="LightGrey">
+          <color rgba="0.8 0.8 0.8 1.0"/>
+        </material>
+    </visual>
+      <collision>
+        <geometry>
+          <mesh filename="package://ur_description/meshes/ur3/visual/osd.stl"/>
+        </geometry>
+        <origin rpy="0 0 0" xyz="-0.015 0.135 0"/>
+        </collision>
+    </link>
+    -->
     <joint name="${prefix}force_jyoint" type="fixed">
       <parent link="${prefix}wrist_3_link" />

File: universal_robot/ur_description/urdf/ur3_joint_limited_robot.urdf.xacro (robot description, xacro)
@@ -6,5 +6,6 @@
   <!-- ur3 -->
   <xacro:include filename="$(find ur_description)/urdf/ur3.urdf.xacro" />
-    <xacro:include filename="$(find realsense2_description)/urdf/test_d415_camera.urdf.xacro" />
+  <!-- realsense_model -->
+  <xacro:include filename="$(find realsense2_description)/urdf/test_d415_camera.urdf.xacro" />
   <!-- arm -->
   <xacro:ur3_robot prefix="" joint_limited="true"
@@ -22,5 +23,5 @@
     <origin xyz="0.0 0.0 0.04" rpy="0.0 0.0 0.0" />
   </joint>
-      <joint name="ommc_joint" type="fixed">
+        <joint name="ommc_joint" type="fixed">
       <parent link="world" />
       <child link = "thin_link" />
